File: KiCad/MZ-700_SD+NRF.kicad_pcb (KiCad board)
At the start: 2 copper layers, 82 x 145 mm, 29 parts, among them J1 MZ-80K BUS, J2 Micro_SD_Card_Kit, J3 INT VCC, J4 EXT 5V, J5 MicroSD Card Adapter, J6 RP2350B Left, J7 RP2350B Right, J8 VGA, J9 Conn_Coaxial, SW1 SW_Push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

Commit message: Add files via upload
Parts:
- C2: value 0.1uF -> 0.01uF
- moved C1 30.8 mm to (109.1, 40.1), turned to 0 degrees
- moved U1 25.4 mm to (106.5, 43.3), turned to 0 degrees
- moved C2 24.8 mm to (92.7, 30.5), turned to 90 degrees
- moved R4 24.8 mm to (97.1, 25.4)
- moved C5 19.8 mm to (109.1, 64.9), turned to 0 degrees
- moved U6 15.2 mm to (106.5, 68.0), turned to 0 degrees
- moved J2 5.00 mm to (134.7, 60.5)
- moved J5 5.00 mm to (126.6, 44.0)
- moved MH2 5.00 mm to (159.6, 149.9)
- moved MH3 5.00 mm to (159.6, 14.9)
- moved SW1 5.00 mm to (149.2, 33.9)
- moved SW2 5.00 mm to (149.2, 23.4)
- moved U4 5.00 mm to (152.4, 66.0)
- moved C6 4.00 mm to (140.9, 22.8)
- moved J4 3.56 mm to (124.8, 33.0)
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Connections:
- J7 pad 4: Net-(C2-Pad2) -> Net-(J7-Pad4)
- J9 pad 1: Net-(J9-Pad1) -> Net-(C2-Pad2)
- R4 pad 1: Net-(J9-Pad1) -> Net-(C2-Pad2)
- R4 pad 2: Net-(C2-Pad2) -> Net-(J7-Pad4)
Routing:
- net Net-(J7-Pad4): track 0.00 -> 208.3 mm, vias 0 -> 1
- net Net-(C2-Pad2): track 130.4 -> 15.0 mm, vias 1 -> 0
- net GND: track 481.0 -> 445.3 mm
- net /~RD: track 169.4 -> 133.9 mm, vias 1 -> 0
- net Net-(J9-Pad1): track 35.5 -> 0.00 mm
- net /A2: track 82.2 -> 115.5 mm, vias 2 -> 1
- net Net-(U1-Pad10): track 6.14 -> 28.4 mm
- net /A6: track 98.8 -> 77.5 mm, vias 0 -> 1
- net /~WR: track 151.4 -> 130.3 mm
- net Net-(U3-Pad22): track 72.4 -> 54.0 mm, vias 1 -> 2
- net /RESET: track 143.4 -> 161.2 mm, vias 2 -> 0
- net Net-(U1-Pad12): track 13.1 -> 30.4 mm
- net Net-(U3-Pad6): track 49.8 -> 32.8 mm
- net +5V: track 193.6 -> 210.4 mm
- net /D2: track 81.8 -> 66.5 mm
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Other:
- board size 82 x 145 mm -> 77 x 145 mm
- board text added: "0.01uF"
- board text added: "MZ-700 SD+NiseRamFile Rev1.5"
- board text removed: "MZ-700 SD+NiseRamFile Rev1.2"

Commit message: Add files via upload
Parts:
- added D1: 1N5819, Diode_THT:D_DO-41_SOD81_P10.16mm_Horizontal, F.Cu at (159.3, 116.3)
Connections:
- J6 pad 1: +5V -> (no net)
- J6 pad 16: (no net) -> Net-(D1-Pad1)
Routing:
- net Net-(D1-Pad1): track 0.00 -> 7.39 mm
- net +5V: track 210.4 -> 205.8 mm
Other:
- board text added: "1N5819"
- board text added: "MZ-700 SD+NiseRamFile Rev1.6"
- board text removed: "MZ-700 SD+NiseRamFile Rev1.5"
