File: KiCad/MZ-700_SD+NRF.sch (KiCad schematic (older format))
At the start: 25 parts, among them J1 MZ-80K BUS, J2 Micro_SD_Card_Kit, J3 INT VCC, J4 EXT 5V, J5 MicroSD Card Adapter, J6 RP2350B Left, J7 RP2350B Right, J8 VGA, J9 Conn_Coaxial, SW1 SW_Push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

Commit message: Add files via upload
Parts:
- C2: value 0.1uF -> 0.01uF
Connections:
- net at J7.4 (Pin_4), R4.2: no longer C2.2
- net at J9.1 (In), R4.1: now also C2.2
Other:
- moved on the sheet: C2
Changed lines of the file:
@@
 encoding utf-8
 Sheet 1 1
-Title "MZ-700_SD"
+Title "MZ-700_SD+NiseRamFile"
 Date "2022-01-14"
-Rev "Rev1.6"
+Rev "Rev1.5"
 Comp ""
 Comment1 ""
@@
 	14600 5850 14750 5850
 Wire Wire Line
-	14300 5850 14100 5850
-Wire Wire Line
 	12550 7100 12250 7100
 $Comp
 L Device:C C2
 U 1 1 69CE90A8
-P 14100 6200
-F 0 "C2" V 13950 6300 50  0000 C CNN
-F 1 "0.1uF" V 13950 6050 50  0000 C CNN
-F 2 "Capacitor_THT:C_Rect_L4.0mm_W2.5mm_P2.50mm" H 14138 6050 50  0001 C CNN
-F 3 "~" H 14100 6200 50  0001 C CNN
-	1    14100 6200
+P 14600 6200
+F 0 "C2" V 14450 6300 50  0000 C CNN
+F 1 "0.01uF" V 14450 6050 50  0000 C CNN
+F 2 "Capacitor_THT:C_Rect_L4.0mm_W2.5mm_P2.50mm" H 14638 6050 50  0001 C CNN
+F 3 "~" H 14600 6200 50  0001 C CNN
+	1    14600 6200
 	-1   0    0    1
 $EndComp
 Wire Wire Line
-	14100 6050 14100 5850
-Connection ~ 14100 5850
-Wire Wire Line
-	14100 6350 14100 6450
-Wire Wire Line
-	14100 6450 14950 6450
+	14600 6050 14600 5850
+Wire Wire Line
+	14600 6350 14600 6450
 Connection ~ 14950 6450
 Wire Wire Line
@@
 Wire Wire Line
 	13450 8200 13050 8200
-Wire Wire Line
-	12250 5850 14100 5850
 Wire Wire Line
 	12250 5850 12250 7100
@@
 	13200 4700 14750 4700
 NoConn ~ 13050 7500
+Wire Wire Line
+	14600 6450 14950 6450
+Wire Wire Line
+	12250 5850 14300 5850
+Connection ~ 14600 5850
 $EndSCHEMATC

Commit message: Add files via upload
Parts:
- added D1: 1N5819, Diode_THT:D_DO-41_SOD81_P10.16mm_Horizontal, symbol Device:D
Connections:
- net +5V: now also D1.2 (A); no longer J6.1 (Pin_1)
- net at J6.16 (Pin_16): now also D1.1 (K)
Changed lines of the file:
@@
 Title "MZ-700_SD+NiseRamFile"
 Date "2022-01-14"
-Rev "Rev1.5"
+Rev "Rev1.6"
 Comp ""
 Comment1 ""
@@
 $EndComp
 Wire Wire Line
-	10450 6800 10050 6800
-Text Label 10050 6800 0    50   ~ 0
+	11650 6800 11250 6800
+Text Label 11500 6800 0    50   ~ 0
 +5V
 Text Label 10050 7200 0    50   ~ 0
@@
 	10050 8200 10450 8200
 NoConn ~ 10450 7000
-NoConn ~ 10950 6800
 NoConn ~ 12550 7000
 NoConn ~ 12550 7300
@@
 	12250 5850 14300 5850
 Connection ~ 14600 5850
+NoConn ~ 10450 6800
+$Comp
+L Device:D D1
+U 1 1 6A1E0307
+P 11100 6800
+F 0 "D1" H 11100 7017 50  0000 C CNN
+F 1 "1N5819" H 11150 6900 50  0000 C CNN
+F 2 "Diode_THT:D_DO-41_SOD81_P10.16mm_Horizontal" H 11100 6800 50  0001 C CNN
+F 3 "~" H 11100 6800 50  0001 C CNN
+	1    11100 6800
+	1    0    0    -1
+$EndComp
 $EndSCHEMATC
